File: HW_design/kicad_soundcard_dev_v0/kicad_soundcard_dev_v0/_autosave-kicad_soundcard_dev_v0.kicad_pcb (KiCad board)
At the start: 4 copper layers, 89 x 51 mm, 141 parts, among them J101 USB_C_Receptacle_USB2.0_16P, J201 DM3AT-SF-PEJM5, J202 1x6P 2.54mm SMD, J203 1x6P 2.54mm SMD, J204 BM04B-SRSS-TB, J205 BM04B-SRSS-TB, J206 BM04B-SRSS-TB, J401 PJ31060-I, J402 PJ31060-I, Q201 L8050QLT1G, Q202 L8050QLT1G, Q401 BSS138LT3G, Q402 BSS138LT3G, SW201 PTS636, SW202 PTS636, U101 AMS1117-3.3, U102 AMS1117-3.3, U201 ESP32-C6-MINI-1/U, U301 LSM6DSL, U302 ICP20100, U401 ES8388

Commit message: Production JLCPCB V0
Parts:
- U401: footprint Package_DFN_QFN:QFN-28-1EP_4x4mm_P0.4mm_EP2.6x2.6mm -> Package_DFN_QFN:QFN-28-1EP_4x4mm_P0.45mm_EP2.6x2.6mm
- moved SW201 32.7 mm to (177.4, 88.9)
- moved G*** 32.7 mm to (162.4, 106.0)
- moved C104 32.6 mm to (140.4, 88.8)
- moved C201 32.6 mm to (157.7, 73.9)
- moved C204 32.6 mm to (177.9, 73.3)
- moved C207 32.6 mm to (174.7, 108.7)
- moved C304 32.6 mm to (177.7, 101.7)
- moved C306 32.6 mm to (142.7, 102.9)
- moved C401 32.6 mm to (142.4, 104.5)
- moved C404 32.6 mm to (132.3, 100.0)
- moved C405 32.6 mm to (130.9, 101.9)
- moved C408 32.6 mm to (137.8, 98.8)
- moved C410 32.6 mm to (130.0, 104.3)
- moved C417 32.6 mm to (131.7, 110.8)
- moved C421 32.6 mm to (131.7, 113.8)
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Routing:
- net +3.3VA: track 40.8 -> 44.6 mm, vias 3 -> 0
- net /MCU/SDIO_DAT2: track 22.6 -> 23.8 mm
- net +3.3V: track 288.8 -> 287.9 mm
- net I2C_SDA: track 66.5 -> 65.7 mm
- net GND: track 116.3 -> 115.8 mm, vias 91 -> 142
Other:
- board text added: "_1_"
- board text added: "_2_"
- board text added: "_3_"
- board text added: "_4_"
- board text added: "_5_"
- board text added: "_6_"
- board text added: "_rgb_led"
- board text removed: "<led_1/2/3>"
- board text removed: "<led_4/5/6>"
